File: portal_lights.kicad_sch (KiCad schematic)
At the start: 0 parts

Commit message: Updates for release v20230724
Other:
- title: FTDI debug probe -> Ingress portal lights
Changed lines of the file:
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@@
   (paper "A4")
   (title_block
-    (title "FTDI debug probe")
+    (title "Ingress portal lights")
     (date "2023-07-19")
   )
