File: pcb/lights.kicad_sch (KiCad schematic)
At the start: 25 parts

Commit message: pcb: Some notes about incorrect RGB LED footprint and connection
Parts:
- LED1, LED10, LED4, LED7: value ASMB-MTB1-0A3A2 -> ASMB-MTB1-0A3A2 (reversed!!!)
Other:
- note added: "LED part # does not match footprint LED footprint is reversed RGB connections are wrong"
Changed lines of the file:
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@@
     (stroke (width 0) (type default))
+  )
+  (text "LED part # does not match footprint\nLED footprint is reversed\nRGB connections are wrong"
+    (at 208.28 68.58 0)
+    (effects (font (size 1.27 1.27)) (justify left bottom))
   )
   (hierarchical_label "R2" (shape input) (at 149.86 58.42 0) (fields_autoplaced)
@@
       (effects (font (size 1.27 1.27)) (justify left))
     )
-    (property "Value" "ASMB-MTB1-0A3A2" (at 207.01 109.22 0)
+    (property "Value" "ASMB-MTB1-0A3A2 (reversed!!!)" (at 207.01 109.22 0)
       (effects (font (size 1.27 1.27)) (justify left))
     )
@@
       (effects (font (size 1.27 1.27)) (justify left))
     )
-    (property "Value" "ASMB-MTB1-0A3A2" (at 207.01 73.66 0)
+    (property "Value" "ASMB-MTB1-0A3A2 (reversed!!!)" (at 207.01 73.66 0)
       (effects (font (size 1.27 1.27)) (justify left))
     )
@@
       (effects (font (size 1.27 1.27)) (justify left))
     )
-    (property "Value" "ASMB-MTB1-0A3A2" (at 207.01 127 0)
+    (property "Value" "ASMB-MTB1-0A3A2 (reversed!!!)" (at 207.01 127 0)
       (effects (font (size 1.27 1.27)) (justify left))
     )
@@
       (effects (font (size 1.27 1.27)) (justify left))
     )
-    (property "Value" "ASMB-MTB1-0A3A2" (at 207.01 91.44 0)
-      (effects (font (size 1.27 1.27)) (justify left))
-    )
+    (property "Value" "ASMB-MTB1-0A3A2 (reversed!!!)" (at 207.01 91.44 0)
+      (effects (font (size 1.27 1.27)) (justify left))
+    )
